File: Kicad 8/Kicad 8/Kicad 8.kicad_pcb (KiCad board)
At the start: 2 copper layers, 93.5 x 99 mm, 14 parts, among them J1 Conn_01x08_Pin - R, J2 Conn_01x08_Pin - L, J3 Conn_01x08_Pin - L, J4 Conn_01x08_Pin - R, J5 Conn_01x05_Pin - 5v, J6 Conn_01x05_Pin - 3.3v, J7 Conn_01x05_Pin - G, SW1 SW_Push, U1 WeMos_D1_mini, U2 WeMos_D1_mini, U3 WeMos_D1_mini, U4 WeMos_D1_mini

Commit message: pcb
Parts:
- D1: footprint LED_THT:LED_D5.0mm -> LED_THT:LED_D3.0mm
- J2: footprint TerminalBlock_RND:TerminalBlock_RND_205-00018_1x08_P5.00mm_Horizontal -> Connector_PinHeader_2.54mm:PinHeader_1x08_P2.54mm_Vertical
- J3: footprint Connector_PinHeader_2.54mm:PinHeader_1x08_P2.54mm_Vertical -> TerminalBlock_RND:TerminalBlock_RND_205-00018_1x08_P5.00mm_Horizontal
- J5, J6, J7: footprint Connector_PinHeader_2.54mm:PinHeader_1x05_P2.54mm_Vertical -> Connector_PinSocket_2.54mm:PinSocket_1x05_P2.54mm_Vertical
- R1: footprint Resistor_THT:R_Axial_DIN0204_L3.6mm_D1.6mm_P5.08mm_Horizontal -> Resistor_THT:R_Axial_DIN0207_L6.3mm_D2.5mm_P7.62mm_Horizontal
- moved D1 137.5 mm to (156.7, 30.0)
- moved R1 135.6 mm to (158.0, 35.2), turned to -90 degrees
- moved SW1 98.6 mm to (83.0, 85.5), turned to 90 degrees
- moved J3 87.6 mm to (174.0, 78.5), turned to -90 degrees
- moved J7 87.5 mm to (160.5, 48.0), turned to 0 degrees
- moved J2 79.5 mm to (88.0, 94.5), turned to 0 degrees
- moved J6 76.5 mm to (160.5, 64.7), turned to 0 degrees
- moved J5 65.6 mm to (160.5, 81.4), turned to 0 degrees
- moved U4 45.7 mm to (131.5, 54.0)
- moved U3 45.7 mm to (93.5, 54.0)
- moved J1 34.2 mm to (122.0, 94.5)
- moved U1 34.2 mm to (93.5, 94.5)
- moved U2 34.1 mm to (131.5, 94.5)
- moved J4 18.2 mm to (174.0, 36.5)
Connections:
- net Net-(D1-K) renamed GND
Routing:
- net GND: track 0.00 -> 232.3 mm
- net Net-(J2-Pin_8): track 0.00 -> 209.9 mm
- net Net-(J2-Pin_3): track 0.00 -> 186.9 mm, vias 0 -> 1
- net Net-(J2-Pin_2): track 0.00 -> 179.0 mm
- net Net-(J1-Pin_8): track 0.00 -> 177.4 mm
- net Net-(J2-Pin_4): track 0.00 -> 176.2 mm
- net Net-(J2-Pin_1): track 0.00 -> 176.0 mm
- net Net-(J2-Pin_7): track 0.00 -> 175.6 mm
- net Net-(J2-Pin_5): track 0.00 -> 174.0 mm
- net Net-(J2-Pin_6): track 0.00 -> 172.3 mm
- net Net-(J1-Pin_3): track 0.00 -> 157.7 mm
- net Net-(J1-Pin_4): track 0.00 -> 155.3 mm
- net Net-(J1-Pin_2): track 0.00 -> 153.7 mm
- net Net-(J1-Pin_5): track 0.00 -> 151.9 mm
- net Net-(J1-Pin_1): track 0.00 -> 150.7 mm
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- added copper zone on B.Cu, net GND
- added copper zone on F.Cu, net GND
Other:
- board size 93.5 x 99 mm -> 99 x 98 mm
- board text added: "3.3v"
- board text added: "Project by AnotherMaker https://github.com/mudmin/AnotherMaker/"
- board text added: "WeMos D1 Max"
- board text removed: "3v3"
